File: Circuits/MPU/SlowShaper.kicad_sch (KiCad schematic)
At the start: 33 parts, among them U10 ADA4805-2ARMZ, U11 ADA4805-2ARMZ

Commit message: Passes DRC
Parts:
- removed R61: 100, Resistor_SMD:R_0603_1608Metric, symbol QuERI_symbols:Rlowp
- added C91: 4.3nF, Capacitor_SMD:C_0603_1608Metric, symbol QuERI_symbols:Csmall
- added R123: 100, Resistor_SMD:R_0603_1608Metric, symbol QuERI_symbols:Rlowp
- C100: renamed from C39; value 11pF -> 750pF
- C101: renamed from C40; value 68pF -> 10nF
- C102: renamed from C41; value 200pF -> 10nF
- C93: renamed from C32; value 20pF -> 1.3nF
- C95: renamed from C34; value 130pF -> 9.1nF
- C98: renamed from C37; value 300pF -> 3.3nF
- C99: renamed from C38; value 11pF -> 750pF
- R133: renamed from R71; value 150 -> 22.1
- R135: renamed from R73; value 499 -> 332
- R136: renamed from R74; value 332 -> 249
- renumbered C31 to C92, C33 to C94, C35 to C96, C36 to C97, D5 to D21, D6 to D22, R62 to R124, R63 to R125, R64 to R126, R65 to R127, R66 to R128, R67 to R129, R68 to R130, R69 to R131, R70 to R132, R72 to R134, R75 to R137, R76 to R138, R77 to R139, R78 to R140, U10 to U22, U11 to U23
Connections:
- net IN: now also R123.1
- net at D21.2 (A), D22.1 (K), R124.1: now also C91.2
- new net: C91.1, R123.2
