File: Circuits/MPU/bypass.kicad_sch (KiCad schematic)
At the start: 63 parts, among them U1 ProASIC

Commit message: Passes DRC
Parts:
- renumbered C201 to C145, C202 to C146, C203 to C147, C204 to C148, C205 to C149, C206 to C150, C207 to C151, C208 to C152, C209 to C153, C210 to C154, C211 to C155, C212 to C156, C213 to C157, C214 to C158, C215 to C159, C216 to C160, C169 to C161, C170 to C162, C185 to C163, C186 to C164, C217 to C165, C218 to C166, C219 to C167, C220 to C168, C171 to C169, C172 to C170, C187 to C171, C188 to C172, C221 to C173, C222 to C174, C223 to C175, C224 to C176, C173 to C177, C174 to C178, C189 to C179, C190 to C180, C175 to C181, C176 to C182, C191 to C183, C192 to C184, C177 to C185, C178 to C186, C193 to C187, C194 to C188, C179 to C189, C180 to C190, C195 to C191, C196 to C192, C181 to C193, C182 to C194, C197 to C195, C198 to C196, C183 to C197, C184 to C198, C163 to C201, C166 to C202, C164 to C203, C167 to C204, C165 to C205, C168 to C206

Commit message: bunch of little fixes
Parts:
- U1: footprint Package_BGA:BGA-484_23.0x23.0mm_Layout22x22_P1.0mm -> Package_BGA:BGA-484_23.0x23.0mm_Layout22x22_P1.0mm
Changed lines of the file:
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@@
 	(title_block
 		(title "QuERI MPU")
-		(date "2024-03-28")
+		(date "2024-05-26")
 		(rev "Draft")
 		(company "Noqsi Aerospace Ltd")
@@
 			)
 		)
-		(property "Footprint" "	Package_BGA:BGA-484_23.0x23.0mm_Layout22x22_P1.0mm"
+		(property "Footprint" "Package_BGA:BGA-484_23.0x23.0mm_Layout22x22_P1.0mm"
 			(at 245.11 22.86 0)
 			(effects
@@
 			)
 		)
-		(property "Footprint" "	Package_BGA:BGA-484_23.0x23.0mm_Layout22x22_P1.0mm"
+		(property "Footprint" "Package_BGA:BGA-484_23.0x23.0mm_Layout22x22_P1.0mm"
 			(at 204.47 95.25 0)
 			(effects
@@
 			)
 		)
-		(property "Footprint" "	Package_BGA:BGA-484_23.0x23.0mm_Layout22x22_P1.0mm"
+		(property "Footprint" "Package_BGA:BGA-484_23.0x23.0mm_Layout22x22_P1.0mm"
 			(at 44.45 95.25 0)
 			(effects
@@
 			)
 		)
-		(property "Footprint" "	Package_BGA:BGA-484_23.0x23.0mm_Layout22x22_P1.0mm"
+		(property "Footprint" "Package_BGA:BGA-484_23.0x23.0mm_Layout22x22_P1.0mm"
 			(at 140.97 22.86 0)
 			(effects
