File: Circuits/MPU/bypass.kicad_sch (KiCad schematic)
At the start: 63 parts, among them U1 ProASIC

Commit message: LVDS I/F for HV
Parts:
- U1: desc FPGA -> FPGA; manf# (none) -> A3PE3000-FGG484
Changed lines of the file:
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@@
 			)
 		)
-		(property "Datasheet" "	https://www.microsemi.com/document-portal/doc_download/130701-ds0098-proasic3e-flash-family-fpgas-datasheet"
+		(property "Datasheet" "https://www.microsemi.com/document-portal/doc_download/130701-ds0098-proasic3e-flash-family-fpgas-datasheet"
 			(at 245.11 27.94 0)
 			(effects
@@
 			)
 		)
-		(property "desc" "	FPGA"
+		(property "desc" "FPGA"
 			(at 245.11 30.48 0)
 			(effects
@@
 			)
 		)
+		(property "manf#" "A3PE3000-FGG484"
+			(at 245.11 25.4 0)
+			(effects
+				(font
+					(size 1.27 1.27)
+				)
+				(justify left)
+				(hide yes)
+			)
+		)
 		(pin "A8"
 		)
@@
 		(pin "A4"
 		)
+		(pin "P19"
+		)
+		(pin "P21"
+		)
+		(pin "R19"
+		)
+		(pin "R21"
+		)
+		(pin "T20"
+		)
+		(pin "T21"
+		)
+		(pin "U20"
+		)
+		(pin "U21"
+		)
+		(pin "V21"
+		)
+		(pin "W21"
+		)
 		(instances
 			(project "MPU"
@@
 			)
 		)
-		(property "Datasheet" "	https://www.microsemi.com/document-portal/doc_download/130701-ds0098-proasic3e-flash-family-fpgas-datasheet"
+		(property "Datasheet" "https://www.microsemi.com/document-portal/doc_download/130701-ds0098-proasic3e-flash-family-fpgas-datasheet"
 			(at 204.47 100.33 0)
 			(effects
@@
 			)
 		)
-		(property "desc" "	FPGA"
+		(property "desc" "FPGA"
 			(at 204.47 102.87 0)
 			(effects
@@
 			)
 		)
+		(property "manf#" "A3PE3000-FGG484"
+			(at 204.47 97.79 0)
+			(effects
+				(font
+					(size 1.27 1.27)
+				)
+				(justify left)
+				(hide yes)
+			)
+		)
 		(pin "A14"
 		)
@@
 		(pin "A15"
 		)
+		(pin "P19"
+		)
+		(pin "P21"
+		)
+		(pin "R19"
+		)
+		(pin "R21"
+		)
+		(pin "T20"
+		)
+		(pin "T21"
+		)
+		(pin "U20"
+		)
+		(pin "U21"
+		)
+		(pin "V21"
+		)
+		(pin "W21"
+		)
 		(instances
 			(project "MPU"
@@
 			)
 		)
-		(property "Datasheet" "	https://www.microsemi.com/document-portal/doc_download/130701-ds0098-proasic3e-flash-family-fpgas-datasheet"
+		(property "Datasheet" "https://www.microsemi.com/document-portal/doc_download/130701-ds0098-proasic3e-flash-family-fpgas-datasheet"
 			(at 44.45 100.33 0)
 			(effects
@@
 			)
 		)
-		(property "desc" "	FPGA"
+		(property "desc" "FPGA"
 			(at 44.45 102.87 0)
 			(effects
@@
 			)
 		)
+		(property "manf#" "A3PE3000-FGG484"
+			(at 44.45 97.79 0)
+			(effects
+				(font
+					(size 1.27 1.27)
+				)
+				(justify left)
+				(hide yes)
+			)
+		)
 		(pin "A14"
 		)
@@
 		(pin "A15"
 		)
+		(pin "P19"
+		)
+		(pin "P21"
+		)
+		(pin "R19"
+		)
+		(pin "R21"
+		)
+		(pin "T20"
+		)
+		(pin "T21"
+		)
+		(pin "U20"
+		)
+		(pin "U21"
+		)
+		(pin "V21"
+		)
+		(pin "W21"
+		)
 		(instances
 			(project "MPU"
@@
 			)
 		)
-		(property "Datasheet" "	https://www.microsemi.com/document-portal/doc_download/130701-ds0098-proasic3e-flash-family-fpgas-datasheet"
+		(property "Datasheet" "https://www.microsemi.com/document-portal/doc_download/130701-ds0098-proasic3e-flash-family-fpgas-datasheet"
 			(at 140.97 27.94 0)
 			(effects
@@
 			)
 		)
-		(property "desc" "	FPGA"
+		(property "desc" "FPGA"
 			(at 140.97 30.48 0)
 			(effects
@@
 			)
 		)
+		(property "manf#" "A3PE3000-FGG484"
+			(at 140.97 25.4 0)
+			(effects
+				(font
+					(size 1.27 1.27)
+				)
+				(justify left)
+				(hide yes)
+			)
+		)
 		(pin "A14"
 		)
@@
 		(pin "A15"
 		)
+		(pin "P19"
+		)
+		(pin "P21"
+		)
+		(pin "R19"
+		)
+		(pin "R21"
+		)
+		(pin "T20"
+		)
+		(pin "T21"
+		)
+		(pin "U20"
+		)
+		(pin "U21"
+		)
+		(pin "V21"
+		)
+		(pin "W21"
+		)
 		(instances
