File: Circuits/MPU/PerFPM.kicad_sch (KiCad schematic)
At the start: 12 parts, among them U1 ADA4805-2ARMZ, U4 LT1715

Commit message: more transcription
Parts:
- added C81: 22uF, Capacitor_SMD:C_1210_3225Metric, symbol QuERI_symbols:C
- added C83: 0.1uF, Capacitor_SMD:C_0603_1608Metric, symbol QuERI_symbols:Csmall
- added C85, C97: 1uF, Capacitor_SMD:C_0805_2012Metric, symbol QuERI_symbols:C
- added C87, C89: 22nF, Capacitor_SMD:C_1210_3225Metric, symbol QuERI_symbols:C
- added C91, C93: 4.7pF, Capacitor_SMD:C_0603_1608Metric, symbol QuERI_symbols:Csmall
- added C95: 200pF, Capacitor_SMD:C_0603_1608Metric, symbol QuERI_symbols:Csmall
- added L5: 4.7uH, Inductor_SMD:L_1008_2520Metric, symbol Device:L
- added Q1: SI4421DY, Package_SO:SOIC-8_3.9x4.9mm_P1.27mm, symbol Transistor_FET:FDS9435A
- added Q3, Q5: MMBTA92, Package_TO_SOT_SMD:SOT-23, symbol Transistor_BJT:MMBTA92
- added R117: 100, Resistor_SMD:R_0603_1608Metric, symbol QuERI_symbols:Rlowp
- added R119, R131: 44.2k, Resistor_SMD:R_0603_1608Metric, symbol QuERI_symbols:Rlowp
- added R121, R123, R125, R126, R147: 1.0k, Resistor_SMD:R_0603_1608Metric, symbol QuERI_symbols:Rlowp
- added R129: 0.2, Resistor_SMD:R_0805_2012Metric, symbol QuERI_symbols:Rlowp
- added R133, R153: 4.99, Resistor_SMD:R_0603_1608Metric, symbol QuERI_symbols:Rlowp
- added R135, R139, R143: 10k, Resistor_SMD:R_0603_1608Metric, symbol QuERI_symbols:Rlowp
- added R137, R141: 10Meg, Resistor_SMD:R_2010_5025Metric, symbol QuERI_symbols:Rlowp
- added R145, R149: 100k, Resistor_SMD:R_0603_1608Metric, symbol QuERI_symbols:Rlowp
- added R151: 249K, Resistor_SMD:R_0603_1608Metric, symbol QuERI_symbols:Rlowp
- added U22, U24: ADA4805-2ARMZ, Package_SO:MSOP-8_3x3mm_P0.65mm, symbol QuERI_symbols:ADA4805-2ARMZ
Connections:
- net +5V: now also R133.1, R153.1
- net +TEC: now also Q1.5 (D), Q1.6 (D), Q1.7 (D), Q1.8 (D)
- net -HV: now also C87.1, C91.2, R135.2, R141.2
- net -TEC: now also R121.2, R125.1, R129.2
- net GND: now also U1.4 (V-), C81.2, C85.2, C87.2, C89.1, C97.2, Q5.1 (B), R123.2, R126.1, R129.1, R149.1, U22.4 (V-), U24.4 (V-)
- net HVDAC: now also R147.1
- net HVHK: now also C95.2, R151.2, U24.3 (+), U24.7
- net TDAC: now also R119.1
- net TIS: now also R131.2, U22.7
- new net: C91.1, C95.1, R141.1, R151.1, U24.6 (-)
- new net: C93.2, R143.1, R145.2, U24.1
- new net: Q5.2 (E), R143.2
- new net: C93.1, R145.1, R147.2, U24.2 (-)
- new net: C89.2, Q3.3 (C), R137.1, R139.2
- new net: C83.1, R117.1, U22.1
- new net: C83.2, R119.2, R123.1, U22.2 (-)
- new net: R121.1, U22.3 (+)
- new net: R125.2, U22.5 (+)
- new net: Q3.1 (B), Q5.3 (C), R137.2
- new net: Q3.2 (E), R135.1
- new net: C85.1, R133.2, U22.8 (V+)
- new net: R126.2, R131.1, U22.6 (-)
- new net: C97.1, R153.2, U24.8 (V+)
- new net: C81.1, L5.2, Q1.1 (S), Q1.2 (S), Q1.3 (S)
- new net: Q1.4 (G), R117.2
- new net: R149.2, U24.5 (+)
- new net +3.3raw: L5.1
- new net -HVunreg: R139.1
Other:
- note added: "Note Kelvin connectoin to ends of 0.2 ohm sense resistor."
- moved on the sheet: C3, C5, C7, R15, R17, R23, U1C, U4C

Commit message: Passes DRC
Parts:
- C10: renamed from C83; Spec 10WVDC X7R -> 50WVDC C0G
- C11: renamed from C91; Spec 250WVDC C0G -> 50WVDC C0G
- C13: renamed from C89; Spec 500WVDC X7R -> 16WVDC X7R
- C14: renamed from C87; Spec 500WVDC X7R -> 16WVDC X7R
- C9: renamed from C93; Spec 250WVDC C0G -> 50WVDC C0G
- renumbered C81 to C12, C5 to C3, C7 to C4, C3 to C5, C85 to C6, C97 to C7, C95 to C8, L5 to L1, Q5 to Q2, R15 to R11, R23 to R12, R11 to R13, R13 to R14, R17 to R15, R133 to R16, R19 to R17, R153 to R18, R21 to R19, R149 to R20, R151 to R21, R119 to R22, R147 to R23, R145 to R24, R121 to R25, R123 to R26, R117 to R27, R141 to R28, R129 to R29, R125 to R30, R126 to R31, R139 to R32, R131 to R33, R143 to R34, R137 to R35, R135 to R36, U4 to U3, U1 to U4, U24 to U5, U22 to U5, U22 to U6, U24 to U6
Connections:
- net In renamed Pulse

Commit message: bunch of little fixes
Parts:
- C10: Spec 50WVDC C0G -> 50WVDC X7R
- C11: footprint Capacitor_SMD:C_0603_1608Metric -> Capacitor_SMD:C_1210_3225Metric; Spec 50WVDC C0G -> 500WVDC C0G
- C13, C14: Spec 16WVDC X7R -> 500WVDC X7R
- R13: value 5.11k -> 4.99k
Changed lines of the file:
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@@
 	(title_block
 		(title "QuERI MPU")
-		(date "2024-03-28")
+		(date "2024-05-26")
 		(rev "Draft")
 		(company "Noqsi Aerospace Ltd")
@@
 			)
 		)
-		(property "Footprint" "Capacitor_SMD:C_0603_1608Metric"
+		(property "Footprint" "Capacitor_SMD:C_1210_3225Metric"
 			(at 187.96 166.6748 0)
 			(effects
@@
 			)
 		)
-		(property "Spec" "50WVDC C0G"
+		(property "Spec" "500WVDC C0G"
 			(at 184.15 167.64 0)
 			(effects
@@
 			)
 		)
-		(property "Spec" "16WVDC X7R"
+		(property "Spec" "500WVDC X7R"
 			(at 203.2 139.7 0)
 			(effects
@@
 			)
 		)
-		(property "Value" "5.11k"
+		(property "Value" "4.99k"
 			(at 52.07 66.04 0)
 			(effects
@@
 			)
 		)
-		(property "Spec" "16WVDC X7R"
+		(property "Spec" "500WVDC X7R"
 			(at 240.03 157.48 0)
 			(effects
@@
 			)
 		)
-		(property "Spec" "50WVDC C0G"
+		(property "Spec" "50WVDC X7R"
 			(at 171.45 36.83 0)
 			(effects
@@
 			(project "MPU"
 				(path "/a3d8c1ad-4320-4fce-bd93-27782a1083f9/dd62822d-07cb-405d-be36-24fcc5049fb2"
-					(page "9")
+					(page "6")
 				)
 				(path "/a3d8c1ad-4320-4fce-bd93-27782a1083f9/1779a0c4-4e7d-4c72-a255-5f54c542193c"
-					(page "10")
+					(page "11")
 				)
 			)
@@
 			(project "MPU"
 				(path "/a3d8c1ad-4320-4fce-bd93-27782a1083f9/dd62822d-07cb-405d-be36-24fcc5049fb2"
-					(page "11")
+					(page "7")
 				)
 				(path "/a3d8c1ad-4320-4fce-bd93-27782a1083f9/1779a0c4-4e7d-4c72-a255-5f54c542193c"
-					(page "13")
+					(page "12")
 				)
 			)
@@
 			(project "MPU"
 				(path "/a3d8c1ad-4320-4fce-bd93-27782a1083f9/dd62822d-07cb-405d-be36-24fcc5049fb2"
-					(page "12")
+					(page "5")
+				)
+				(path "/a3d8c1ad-4320-4fce-bd93-27782a1083f9/1779a0c4-4e7d-4c72-a255-5f54c542193c"
+					(page "10")
 				)
 			)
@@
 			(project "MPU"
 				(path "/a3d8c1ad-4320-4fce-bd93-27782a1083f9/dd62822d-07cb-405d-be36-24fcc5049fb2"
-					(page "8")
+					(page "4")
+				)
+				(path "/a3d8c1ad-4320-4fce-bd93-27782a1083f9/1779a0c4-4e7d-4c72-a255-5f54c542193c"
+					(page "9")
 				)
 			)

Commit message: Better names
Other:
- sheet FastShaper renamed Fast Shaper
- sheet Pulse Capture renamed Fast Pulse Capture
- sheet Pulse Capture1 renamed Slow Pulse Capture
- sheet SlowShaper renamed Slow Shaper
Changed lines of the file:
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@@
 			(color 0 0 0 0.0000)
 		)
-		(property "Sheetname" "SlowShaper"
+		(property "Sheetname" "Slow Shaper"
 			(at 68.58 48.8184 0)
 			(effects
@@
 			(color 0 0 0 0.0000)
 		)
-		(property "Sheetname" "Pulse Capture1"
+		(property "Sheetname" "Slow Pulse Capture"
 			(at 95.25 47.5484 0)
 			(effects
@@
 			(color 0 0 0 0.0000)
 		)
-		(property "Sheetname" "Pulse Capture"
+		(property "Sheetname" "Fast Pulse Capture"
 			(at 95.25 23.4184 0)
 			(effects
@@
 			(color 0 0 0 0.0000)
 		)
-		(property "Sheetname" "FastShaper"
+		(property "Sheetname" "Fast Shaper"
 			(at 68.58 24.6884 0)
 			(effects
