File: Circuits/MPU/FastCapture.kicad_sch (KiCad schematic)
At the start: 41 parts, among them U16 MAX4636EUB, U29 CD74AC00M96, U31 LT1715, U37 LT1715, U38 ADA4805-2ARMZ, U39 AD7984BRMZ, U41 CD74AC00M96, U9 ADA4805-2ARMZ

Commit message: Simplify fast capture logic
Parts:
- removed C70: 1uF, Capacitor_SMD:C_0805_2012Metric, symbol QuERI_symbols:C
- removed R77: 200, Resistor_SMD:R_0603_1608Metric, symbol QuERI_symbols:Rlowp
- removed U41: CD74AC00M96, Package_SO:SOIC-14_3.9x8.7mm_P1.27mm, symbol QuERI:74AC00
Connections:
- net GND: now also U29.1, U29.2
- net LLD: now also U31.3 (-); no longer U31.4 (+)
- net ~{TRACK}: no longer U29.5
- net at U31.7: now also U29.4; no longer U29.1
- net at U29.6: now also U29.9; no longer U29.2
- net at U29.3: no longer U29.4
- net at R212.1, R50.1, U38.1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: now also U31.4 (+); no longer U31.3 (-)
- net at R219.2, U37.8: now also U29.5
Other:
- moved on the sheet: C225, R217, R219, U31B, U37A
