File: Circuits/MPU/SerialIF.kicad_sch (KiCad schematic)
At the start: 24 parts, among them Q13 SSM3K345R, U1 ProASIC, U2 ADM3488ARZ, U40 ADM3488ARZ, X1 KC2016K50.0000C1GE00

Commit message: Fix symbols for release
Parts:
- X1: footprint Crystal:Crystal_SMD_2016-4Pin_2.0x1.6mm -> Oscillator:Oscillator_SMD_SeikoEpson_SG210-4Pin_2.5x2.0mm
Changed lines of the file:
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@@
 			)
 		)
-		(property "Description" "	A3PE3000-FGG484"
+		(property "Description" "A3PE3000-FGG484"
 			(at 120.65 176.53 0)
 			(effects
@@
 			)
 		)
-		(property "Footprint" "Crystal:Crystal_SMD_2016-4Pin_2.0x1.6mm"
+		(property "Footprint" "Oscillator:Oscillator_SMD_SeikoEpson_SG210-4Pin_2.5x2.0mm"
 			(at 167.64 120.65 0)
 			(effects
@@
 			)
 		)
-		(property "Description" "	A3PE3000-FGG484"
+		(property "Description" "A3PE3000-FGG484"
 			(at 167.64 63.5 0)
 			(effects
