File: Circuits/MPU/MPU.kicad_sch (KiCad schematic)
At the start: 13 parts, among them J1 5-1814400-1, J10 Conn_02x10_Odd_Even, J13 MDM15_Plug, J2 5-1814400-1, J3 MDM9_Plug, J4 MDM9_Plug, J5 0010085031, J6 MDM9_Receptacle, J8 Conn_02x05_Odd_Even, U1 ProASIC

Commit message: add missing footprints
Parts:
- J13: footprint (none) -> MDM-15PCBR:ITT_MDM-15PCBR
- J3, J4, J6: footprint (none) -> MDM-9SCBRP:ITT_MDM-9SCBRP
- J5: footprint (none) -> Connector_Molex:Molex_KK-396_A-41791-0003_1x03_P3.96mm_Vertical
Changed lines of the file:
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@@
 			)
 		)
-		(property "Footprint" ""
+		(property "Footprint" "MDM-9SCBRP:ITT_MDM-9SCBRP"
 			(at 30.48 130.81 0)
 			(effects
@@
 			)
 		)
-		(property "Footprint" ""
+		(property "Footprint" "MDM-9SCBRP:ITT_MDM-9SCBRP"
 			(at 30.48 54.61 0)
 			(effects
@@
 			)
 		)
-		(property "Footprint" ""
+		(property "Footprint" "Connector_Molex:Molex_KK-396_A-41791-0003_1x03_P3.96mm_Vertical"
 			(at 116.84 163.83 0)
 			(effects
@@
 			)
 		)
-		(property "Footprint" ""
+		(property "Footprint" "MDM-15PCBR:ITT_MDM-15PCBR"
 			(at 165.1 107.95 0)
 			(effects
@@
 			)
 		)
-		(property "Footprint" ""
+		(property "Footprint" "MDM-9SCBRP:ITT_MDM-9SCBRP"
 			(at 161.29 29.21 0)
 			(effects

Commit message: PCB layout from Joel
Connections:
- net PerFPM-0/Pulse: now also J1.5; no longer J1.2
- net PerFPM-1/Pulse: now also J2.5; no longer J2.2
Changed lines of the file:
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@@
 		(fields_autoplaced yes)
 		(property "Reference" "J2"
-			(at 27.9399 102.87 0)
+			(at 27.9394 102.87 0)
 			(effects
 				(font
@@
 		)
 		(property "Value" "5-1814400-1"
-			(at 27.9399 105.41 0)
+			(at 27.9394 105.41 0)
 			(effects
 				(font
@@
 		(pin "1"
 		)
-		(pin "2"
+		(pin "5"
 		)
 		(instances
@@
 	)
 	(symbol
+		(lib_name "5-1814400-1_1")
 		(lib_id "dk_Coax:5-1814400-1")
 		(at 27.94 33.02 0)
@@
 		(pin "1"
 		)
-		(pin "2"
+		(pin "5"
 		)
 		(instances
