File: Circuits/MPU/ChainSim/ChainSim.kicad_sch (KiCad schematic)
At the start: 4 parts, among them U3 LT1715, U4 ADA4805-2ARMZ

Commit message: sim snapshot
Parts:
- added V1: 3.3V, symbol Simulation_SPICE:VDC
- added V2, V3: 2.1V, symbol Simulation_SPICE:VDC
- added V4: VPWL, symbol Simulation_SPICE:VPWL
- added V5: 5V, symbol Simulation_SPICE:VDC
- added V6: 2.5v, symbol Simulation_SPICE:VDC
- added V7: 4v, symbol Simulation_SPICE:VDC
- added V8: 2v, symbol Simulation_SPICE:VDC
- renumbered R13 to R1, R14 to R2, U4 to U1, U3 to U2
Connections:
- net +2.5V: now also V6.1
- net FLLD: now also V2.1
- net SLLD: now also V3.1
- net VFS: now also V7.1
- net VHS: now also V8.1
- net at U1.3 (+): now also V4.1
- new net +3.3V: V1.1
- new net +5V: V5.1
- new net GND: V1.2, V2.2, V3.2, V4.2, V5.2, V6.2, V7.2, V8.2
Other:
- note added: ".options gmin=1e-10 .options abstol=1e-10 .options reltol=0.1"
- moved on the sheet: R1, R2, U1A, U1B, U2A, U2B

Commit message: trying to get a stable sim
Other:
- note added: ".options gmin=1e-9 .options abstol=1e-9 .options reltol=0.1 .options vntol=1e-4"
- note removed: ".options gmin=1e-10 .options abstol=1e-10 .options reltol=0.1"
Changed lines of the file:
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@@
+	)
+	(junction
+		(at 102.87 49.53)
+		(diameter 0)
+		(color 0 0 0 0)
 	)
 	(junction
@@
 	(wire
 		(pts
-			(xy 99.06 49.53) (xy 113.03 49.53)
+			(xy 99.06 49.53) (xy 102.87 49.53)
 		)
 		(stroke
@@
 	(wire
 		(pts
+			(xy 102.87 49.53) (xy 113.03 49.53)
+		)
+		(stroke
+			(width 0)
+			(type default)
+		)
+	)
+	(wire
+		(pts
 			(xy 133.35 45.72) (xy 133.35 43.18)
 		)
@@
 	(wire
 		(pts
+			(xy 102.87 46.99) (xy 102.87 49.53)
+		)
+		(stroke
+			(width 0)
+			(type default)
+		)
+	)
+	(wire
+		(pts
 			(xy 81.28 71.12) (xy 81.28 53.34)
 		)
@@
 	(wire
 		(pts
+			(xy 104.14 46.99) (xy 102.87 46.99)
+		)
+		(stroke
+			(width 0)
+			(type default)
+		)
+	)
+	(wire
+		(pts
 			(xy 104.14 114.3) (xy 109.22 114.3)
 		)
@@
 		)
 	)
-	(text ".options gmin=1e-10\n.options abstol=1e-10\n.options reltol=0.1\n"
+	(text ".options gmin=1e-9\n.options abstol=1e-9\n.options reltol=0.1\n.options vntol=1e-4\n"
 		(exclude_from_sim no)
 		(at 204.216 30.226 0)
@@
 			(effects
 				(font
+					(size 1.27 1.27)
+				)
+				(justify left)
+				(hide yes)
+			)
+		)
+	)
+	(global_label "FU"
+		(shape output)
+		(at 104.14 46.99 0)
+		(fields_autoplaced yes)
+		(effects
+			(font
+				(size 1.27 1.27)
+			)
+			(justify left)
+		)
+		(property "Intersheetrefs" "${INTERSHEET_REFS}"
+			(at 109.5443 46.99 0)
+			(effects
+				(font
