File: Circuits/MPU/ChainSim/SlowShaper.kicad_sch (KiCad schematic)
At the start: 34 parts, among them U22 ADA4805-2ARMZ, U23 ADA4805-2ARMZ

Commit message: sim snapshot
Parts:
- renumbered C91 to C13, C92 to C14, C93 to C15, C94 to C16, C95 to C17, C96 to C18, C97 to C19, C98 to C20, C99 to C21, C100 to C22, C101 to C23, C102 to C24, D21 to D3, D22 to D4, R123 to R21, R124 to R22, R125 to R23, R126 to R24, R127 to R25, R128 to R26, R129 to R27, R130 to R28, R131 to R29, R132 to R30, R133 to R31, R134 to R32, R135 to R33, R136 to R34, R137 to R35, R138 to R36, R139 to R37, R140 to R38, U22 to U5, U23 to U6
